File: hardware/r2.0/mmdvm_hs-hat.sch (KiCad schematic (older format))
At the start: 84 parts, among them P1 I2C, P2 Display, P3 SMA, P4 STLINK, U1 ADF7021, U2 STM32F103C8T6, X1 TCXO, Y1 8MHz

Commit message: Initial routing done for rev2.0
Parts:
- removed C30: 10u/10V, Capacitors_Tantalum_SMD:CP_Tantalum_Case-A_EIA-3216-18_Reflow, symbol mmdvm_hs-hat-rescue:CP-RESCUE-mmdvm_hs-hat
- removed U?: AP1117-33, Package_TO_SOT_SMD:SOT-223-3_TabPin2, symbol Regulator_Linear:AP1117-33
- removed U?: USBLC6-2SC6, Package_TO_SOT_SMD:SOT-23-6, symbol Power_Protection:USBLC6-2SC6
- added U3: TLV70233_SOT23-5, Package_TO_SOT_SMD:SOT-23-5, symbol Regulator_Linear:TLV70233_SOT23-5
- added U4: USBLC6-2, pkl_housings_sot:SOT-23-6, symbol pkl_misc:USBLC6-2
- C1, C10, C11, C12, C13, C14, C15, C17, C18, C19, C2, C20, C21, C22, C23, C24, C25, C26, C27, C28, C29, C3, C4, C5, C6, C7, C8, C9: footprint Capacitors_SMD:C_0402 -> pkl_dipol:C_0402
- C31: footprint Capacitors_SMD:C_0402 -> pkl_dipol:C_0603
- D1, D2, D3, D4, D5, D6, D7, D8, D9: footprint LEDs:LED_0402 -> LED_SMD:LED_0402_1005Metric
- D10: renamed from D?; footprint LEDs:LED_0402 -> LED_SMD:LED_0402_1005Metric
- L1, L2, L3, L4, L5: footprint Inductors_SMD:L_0402 -> pkl_dipol:L_0402
- P1: value I2C -> OLED; footprint Connector_PinHeader_2.54mm:PinHeader_1x04_P2.54mm_Vertical -> pkl_pin_headers:Pin_Header_Straight_1x04
- P2: footprint Connector_PinHeader_2.54mm:PinHeader_1x04_P2.54mm_Vertical -> pkl_pin_headers:Pin_Header_Straight_1x04
- P3: footprint (none) -> Connector_Coaxial:SMA_Amphenol_132291-12_Vertical
- P4: footprint Connector:Tag-Connect_TC2030-IDC-NL_2x03_P1.27mm_Vertical -> pkl_tag_connect:TC2030-NL_SMALL
- R1, R10, R11, R12, R13, R14, R15, R16, R17, R18, R19, R2, R3, R4, R5, R6, R7, R8, R9: footprint Resistors_SMD:R_0402 -> pkl_dipol:R_0402
- R20, R21, R22, R23, R25, R26: renamed from R?; footprint Resistors_SMD:R_0402 -> pkl_dipol:R_0402
- R24: renamed from R?; footprint (none) -> pkl_dipol:R_0402
- Y1: footprint Crystal:Crystal_SMD_Abracon_ABM3-2Pin_5.0x3.2mm -> Crystal:Crystal_SMD_3225-4Pin_3.2x2.5mm; symbol mmdvm_hs-hat-rescue:Crystal-RESCUE-mmdvm_hs-hat -> Device:Crystal_GND24_Small; MFR ABRACON -> ECS; MPN ABM3-8.000MHz-D2Y-T -> ECS-80-18-33-JGN-TR; SPN 815-ABM3-8-D2Y-T -> 520-80-18-33-JGN-TR
- gave numbers to parts that had none: 1
Connections:
- net +5V: now also U4.5 (VBUS); no longer R24.1
- net GND: now also Y1.2, Y1.4, U3.2 (GND), U4.2 (GND)
- net VDD: now also R24.1, U3.5 (OUT)
- net at C23.2, U2.6 (PD1): now also Y1.3; no longer Y1.2
- net at L5.2: now also U3.1 (IN), U3.3 (EN)
- net at R24.2, R26.1: now also U4.4 (IO2)
- net at R25.1: now also U4.6 (IO1)
- net xUSB_DN renamed xUDN
- net xUDN: now also U4.1 (IO1)
- net xUSB_DP renamed xUDP
- net xUDP: now also U4.3 (IO2)
Other:
- note removed: "replace with smaller xtal"
- moved on the sheet: R21, R7

Commit message: Small silk screen changes
Final Revision 2.0, tested and working
Parts:
- U3: symbol Regulator_Linear:TLV70233_SOT23-5 -> mmdvm_hs-hat-rescue:TLV70233_SOT23-5-Regulator_Linear
- Y1: footprint Crystal:Crystal_SMD_3225-4Pin_3.2x2.5mm -> Crystal:Crystal_SMD_5032-2Pin_5.0x3.2mm; symbol Device:Crystal_GND24_Small -> Device:Crystal_Small
Connections:
- net GND: no longer Y1.2, Y1.4
- net at C23.2, U2.6 (PD1): now also Y1.2; no longer Y1.3
Changed lines of the file:
@@
 EESchema Schematic File Version 4
-LIBS:mmdvm_hs-hat-cache
 EELAYER 30 0
 EELAYER END
@@
 $EndComp
 $Comp
-L Device:Crystal_GND24_Small Y1
+L Device:Crystal_Small Y1
 U 1 1 5895F2AD
 P 7800 1950
 F 0 "Y1" H 7650 2100 50  0000 C CNN
 F 1 "8MHz" H 7950 2100 50  0000 C CNN
-F 2 "Crystal:Crystal_SMD_3225-4Pin_3.2x2.5mm" H 7800 1950 50  0001 C CNN
+F 2 "Crystal:Crystal_SMD_5032-2Pin_5.0x3.2mm" H 7800 1950 50  0001 C CNN
 F 3 "" H 7800 1950 50  0001 C CNN
 F 4 "ECS" H 1100 -350 50  0001 C CNN "MFR"
@@
 Wire Wire Line
 	7900 1950 8050 1950
-Wire Wire Line
-	7800 1850 7800 1750
-Wire Wire Line
-	7800 1750 7250 1750
-Wire Wire Line
-	7250 1750 7250 2450
-$Comp
-L power:GND #PWR0101
-U 1 1 5F209A52
-P 7250 2450
-F 0 "#PWR0101" H 7250 2200 50  0001 C CNN
-F 1 "GND" H 7250 2300 50  0000 C CNN
-F 2 "" H 7250 2450 50  0000 C CNN
-F 3 "" H 7250 2450 50  0000 C CNN
-	1    7250 2450
-	1    0    0    -1
-$EndComp
-$Comp
-L power:GND #PWR0108
-U 1 1 5F209E98
-P 7800 2450
-F 0 "#PWR0108" H 7800 2200 50  0001 C CNN
-F 1 "GND" H 7800 2300 50  0000 C CNN
-F 2 "" H 7800 2450 50  0000 C CNN
-F 3 "" H 7800 2450 50  0000 C CNN
-	1    7800 2450
-	1    0    0    -1
-$EndComp
-Wire Wire Line
-	7800 2050 7800 2450
 $Comp
 L power:VDD #PWR039
@@
 $EndComp
 $Comp
-L Regulator_Linear:TLV70233_SOT23-5 U3
+L mmdvm_hs-hat-rescue:TLV70233_SOT23-5-Regulator_Linear U3
 U 1 1 5F1F0AB4
 P 4200 1000
